Commit message: Task 2: Integrate STVL with VLP-16 for 3D dynamic obstacle detection
- Replace voxel_layer with spatio_temporal_voxel_layer in Nav2 costmap
- Configure VLP-16 as STVL observation source (marking + clearing)
- Fix topic namespace using absolute path /a200_1103/sensors/lidar3d_0/points
- Fix TF namespace issue using topic_tools relay nodes
- Local costmap: voxel_decay 5s, Global costmap: voxel_decay 15s
- Both costmaps confirmed active with STVL publishing voxel_grid at 3.5Hz

File: robot.urdf.xacro (robot description, xacro)
@@ -50,9 +50,4 @@
     <origin xyz="0.0 0.0 0.0" rpy="0.0 0.0 0.0"/>
   </xacro:velodyne_lidar>
-  <!-- camera_0 -->
-  <xacro:include filename="$(find clearpath_sensors_description)/urdf/intel_realsense.urdf.xacro"/>
-  <xacro:intel_realsense name="camera_0" parent_link="fath_pivot_0_mount" update_rate="30" image_height="480" image_width="640">
-    <origin xyz="0.0 0.0 0.0" rpy="0.0 0.0 0.0"/>
-  </xacro:intel_realsense>
   <!-- Manipulators -->
   <!-- Extras -->
